Commit message: 修复仿真初始化bug

File: src/401pius/urdf/401pius.urdf (robot description, URDF)
Before this commit: robot 401pius, 6 links, 5 joints
Links:
- added link base_footprint; visual sphere radius=0.001
- link chejia_link: mass 2.42397545608915 -> 2.424
- link youhoulun_Link: mass 0.634778552429949 -> 0.635
- link youqianlun_Link: mass 0.37912408551256 -> 0.379
- link zhuanxiangjia_Link: mass 0.636763996187421 -> 0.637
- link zuohoulun_Link: mass 0.634779873374433 -> 0.635
- link zuoqianlun_Link: mass 0.379124506048444 -> 0.379
Joints:
- added joint chejia_link2base_footprint: type fixed, parent base_footprint, child chejia_link, origin xyz=0 0 0.33

File: src/gazebo/urdf/my_base_camera_laser.xacro (robot description, xacro)
@@ -4,3 +4,6 @@
     <xacro:include filename="my_camera.xacro" />
     <xacro:include filename="my_laser.xacro" />
+    <xacro:include filename="gezebo/move.xacro" />
+    <xacro:include filename="gezebo/laser.xacro" />
+    <xacro:include filename="gezebo/camera.xacro" />
 </robot>

Commit message: 一些更改

File: src/401pius/urdf/401pius.urdf (robot description, URDF)
Before this commit: robot 401pius, 7 links, 6 joints
Links:
- added link laser, mass 0.1; collision cylinder length=0.05 radius=0.03; visual cylinder length=0.05 radius=0.03
Joints:
- added joint laser2chejia_link: type fixed, parent chejia_link, child laser, origin xyz=0.0 0.0 0.0

File: src/segway-401_plus/urdf/segway_e1.urdf (robot description, URDF)
Before this commit: robot segway_e1_description, 7 links, 6 joints
Links:
- removed link Chassis front beam
- removed link Left front wheel
- removed link Left rear wheel
- removed link Right front wheel
- removed link Right rear wheel
- added link Chassis_front_beam, mass 0.48416; collision mesh filename=package://segway_e1_description/meshes/Chassis front beam.S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; visual mesh filename=package://segway_e1_description/meshes/Chassis front beam.S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
- added link Left_front_wheel, mass 1.25; collision mesh filename=package://segway_e1_description/meshes/Wheel.STL; visual mesh filename=package://segway_e1_description/meshes/Wheel.STL
- added link Left_rear_wheel, mass 1.25; collision mesh filename=package://segway_e1_description/meshes/Wheel.STL; visual mesh filename=package://segway_e1_description/meshes/Wheel.STL
- added link Right_front_wheel, mass 1.25; collision mesh filename=package://segway_e1_description/meshes/Wheel.STL; visual mesh filename=package://segway_e1_description/meshes/Wheel.STL
- added link Right_rear_wheel, mass 1.25; collision mesh filename=package://segway_e1_description/meshes/Wheel.STL; visual mesh filename=package://segway_e1_description/meshes/Wheel.STL
- added link base_footprint; visual sphere radius=0.001
- added link laser, mass 0.1; collision cylinder length=0.05 radius=0.03; visual cylinder length=0.05 radius=0.03
- link Chassis body: mass 1.5192 -> 1.5
Joints:
- removed joint Chassis front beam
- removed joint Left front wheel
- removed joint Left rear wheel
- removed joint Right front wheel
- removed joint Right rear wheel
- added joint Chassis_front_beam_joint: type revolute, parent Chassis body, child Chassis_front_beam, origin xyz=-0.0335 0.504 -0.0515 rpy=0 0 0, axis 0 0 1, limit lower=-0.3 upper=0.3 effort=0 velocity=0
- added joint Left_front_wheel_joint: type continuous, parent Chassis_front_beam, child Left_front_wheel, origin xyz=-0.27184 0.0001 -0.028906 rpy=1.5708 0 1.5708, axis 0 0 -1
- added joint Left_rear_wheel_joint: type continuous, parent Chassis body, child Left_rear_wheel, origin xyz=-0.30884 0.04815 -0.080406 rpy=1.5708 0 1.5708, axis 0 0 -1
- added joint Right_front_wheel_joint: type continuous, parent Chassis_front_beam, child Right_front_wheel, origin xyz=0.27184 0.0001 -0.028906 rpy=1.5708 0 1.5708, axis 0 0 -1
- added joint Right_rear_wheel_joint: type continuous, parent Chassis body, child Right_rear_wheel, origin xyz=0.24188 0.04815 -0.080406 rpy=1.5708 0 1.5708, axis 0 0 -1
- added joint base_link2base_footprint: type fixed, parent base_footprint, child base_link, origin xyz=0 0 0.19
- added joint laser2base_link: type fixed, parent base_link, child laser, origin xyz=0.0 0.0 0.12
